File: Hardware/EthernetGCS.sch (EAGLE design)
At the start: 80 parts, among them IC1 PIC24FJ64GA002_QFN, IC3 24AA00OT, J2 HR911105A, Q2 25Mhz, U1 MIC5219-3.3V, U3 MIC5219-3.3V, U4 ENC28J60-QFN, U5 MIC5219-3.3V, U7 FT232RL-BASICSSOP, X2 USB-A-H

Commit message: More layout. Deleting reference board, adding ground planes.
Parts:
- removed C21: 1uF, SparkFun:CAP0402-CAP
- removed C22: 470pF, SparkFun:CAP0402-CAP
- removed C23: 10uF, SparkFun:CAP_POL1206
- removed C24, C25: 0.1uF, SparkFun:CAP0402-CAP
- removed J$2: SMA_EDGE, 3DRobotics:SMA_EDGE
- removed JP3, JP4: FIDUCIAL1X2, SparkFun:FIDUCIAL1X2
- removed L2, L3, L4, L5: BLM15HD102SN1, pel_dipol_comp:INDUCTOR-0402
- removed L7: BKP1005HS121-T, pel_dipol_comp:INDUCTOR-0402
- removed LED3: GREEN, SparkFun:LED0603
- removed LED4: RED, SparkFun:LED0603
- removed R11, R6: 330, SparkFun:RESISTOR0402-RES
- removed U5: MIC5219-3.3V, SparkFun:V_REG_LDOSMD
- removed U6: (no value), 3DRobotics:HM-TRPSMD
- removed U7: FT232RL-BASICSSOP, SparkFun:FT232RL-BASICSSOP
- removed X2: USB-A-H, SparkFun:USB-A-H
Connections:
- removed net CTS1: U6.!CONFIG, U7.CTS
- removed net DTR1: U7.DTR
- removed net N$20: C22.1, U5.BP
- removed net N$21: J$2.SIGNAL, U6.ANT
- removed net N$23: C24.1, U7.3V3OUT, U7.VCCIO
- removed net N$24: U7.USBDP, X2.D-
- removed net N$25: U7.USBDM, X2.D+
- removed net N$26: LED4.A, R11.1
- removed net N$27: LED3.A, R6.1
- removed net N$28: LED4.C, U7.TXLED
- removed net N$29: LED3.C, U7.RXLED
- removed net N$30: L2.2, U6.DTX
- removed net N$31: L3.2, U6.DRX
- removed net N$32: L7.1, X2.GND
- removed net N$4: L4.2, U2.DTX
- removed net N$7: L5.2, U2.DRX
- removed net RTS1: U6.!ENABLE, U7.RTS
- removed net RX1: L3.1, U7.TXD
- removed net TX1: L2.1, U7.RXD
- net 3.3V: no longer C23.+, U5.OUT, U6.VCC
- net 5V: no longer C21.1, C25.1, L7.2, R11.2, R6.2, U5.EN, U5.IN, U7.VCC
- net GND: now also R1.1, R2.1; no longer C21.2, C22.2, C23.-, C24.2, C25.2, J$2.GND@0, J$2.GND@1, J$2.GND@2, J$2.GND@3, LED1.C, LED2.C, U5.GND, U6.AGND, U6.GND, U7.AGND, U7.GND1, U7.GND2, U7.GND3, U7.TEST, X2.VBUS
- net LED_RX: now also LED1.A; no longer R1.2
- net LED_TX: now also LED2.A; no longer R2.2
- net N$8: now also LED1.C, R1.2; no longer LED2.A, R2.1
- net N$9: now also LED2.C, R2.2; no longer LED1.A, R1.1
- net RX: now also U2.DRX; no longer L5.1
- net TX: now also U2.DTX; no longer L4.1
Other:
- note removed: "Power"

Commit message: Layout is finished.
Or at least is seams that way.
Parts:
- removed C11, C8: 0.1uF, SparkFun:CAP0402-CAP
- added JP3: FIDUCIAL1X2, SparkFun:FIDUCIAL1X2
Connections:
- net GND: no longer C11.2, C8.2
- net V+: no longer C11.1, C8.1
Other:
- moved on the sheet: D1, R10, R13
Changed lines of the file:
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@@
 <part name="IC3" library="microchip" deviceset="24*00" device="OT" technology="AA"/>
 <part name="U4" library="microchip-enc28j60" deviceset="ENC28J60-*" device="QFN"/>
-<part name="C8" library="SparkFun" deviceset="CAP" device="0402-CAP" value="0.1uF"/>
 <part name="C9" library="SparkFun" deviceset="CAP" device="0402-CAP" value="0.1uF"/>
 <part name="C10" library="SparkFun" deviceset="CAP" device="0402-CAP" value="0.1uF"/>
-<part name="C11" library="SparkFun" deviceset="CAP" device="0402-CAP" value="0.1uF"/>
 <part name="C12" library="SparkFun" deviceset="CAP" device="0402-CAP" value="0.1uF"/>
 <part name="C13" library="SparkFun" deviceset="CAP" device="0402-CAP" value="0.1uF"/>
@@
 <part name="GND48" library="supply1" deviceset="GND" device=""/>
 <part name="U$8" library="SparkFun" deviceset="5V" device=""/>
+<part name="JP3" library="SparkFun" deviceset="FIDUCIAL" device="1X2"/>
 </parts>
 <sheets>
@@
 <wire x1="175.26" y1="66.04" x2="248.92" y2="66.04" width="0.3048" layer="97"/>
 <wire x1="331.47" y1="100.33" x2="330.9874" y2="99.8474" width="0.254" layer="94"/>
-<wire x1="-36.83" y1="186.6646" x2="-36.83" y2="187.198" width="0.254" layer="94"/>
-<wire x1="-36.83" y1="187.198" x2="-36.2712" y2="187.198" width="0.254" layer="94"/>
-<wire x1="-36.2712" y1="187.198" x2="-36.2712" y2="186.7662" width="0.254" layer="94"/>
 </plain>
 <instances>
@@
 <attribute name="VALUE" x="51.054" y="72.644" size="1.778" layer="96"/>
 </instance>
-<instance part="C8" gate="G$1" x="30.48" y="50.8"/>
 <instance part="C9" gate="G$1" x="40.64" y="50.8"/>
 <instance part="C10" gate="G$1" x="50.8" y="50.8"/>
-<instance part="C11" gate="G$1" x="60.96" y="50.8"/>
 <instance part="C12" gate="G$1" x="109.22" y="134.62" rot="R90"/>
 <instance part="C13" gate="G$1" x="109.22" y="139.7" rot="R90"/>
@@
 </instance>
 <instance part="GND28" gate="1" x="266.7" y="96.52"/>
-<instance part="R10" gate="G$1" x="289.56" y="73.66" smashed="yes">
-<attribute name="NAME" x="282.448" y="74.1426" size="1.778" layer="95"/>
-<attribute name="VALUE" x="292.608" y="71.374" size="1.778" layer="96"/>
-</instance>
-<instance part="R13" gate="G$1" x="289.56" y="71.12" smashed="yes">
-<attribute name="NAME" x="282.448" y="71.6026" size="1.778" layer="95"/>
-<attribute name="VALUE" x="292.608" y="68.834" size="1.778" layer="96"/>
+<instance part="R10" gate="G$1" x="284.48" y="73.66" smashed="yes">
+<attribute name="NAME" x="277.368" y="74.1426" size="1.778" layer="95"/>
+<attribute name="VALUE" x="287.528" y="71.374" size="1.778" layer="96"/>
+</instance>
+<instance part="R13" gate="G$1" x="284.48" y="71.12" smashed="yes">
+<attribute name="NAME" x="277.368" y="71.6026" size="1.778" layer="95"/>
+<attribute name="VALUE" x="287.528" y="68.834" size="1.778" layer="96"/>
 </instance>
 <instance part="GND30" gate="1" x="53.34" y="7.62"/>
@@
 <instance part="GND43" gate="1" x="228.6" y="48.26" rot="R90"/>
 <instance part="GND45" gate="1" x="144.78" y="167.64" rot="MR90"/>
-<instance part="U$4" gate="G$1" x="350.52" y="104.14" rot="R270"/>
-<instance part="GND46" gate="1" x="332.74" y="86.36"/>
+<instance part="U$4" gate="G$1" x="337.82" y="104.14" rot="R270"/>
+<instance part="GND46" gate="1" x="332.74" y="93.98"/>
 <instance part="D4" gate="G$1" x="332.74" y="99.06" smashed="yes" rot="R90">
 <attribute name="NAME" x="335.28" y="96.52" size="1.27" layer="95" rot="R90"/>
-<attribute name="VALUE" x="339.09" y="86.36" size="1.27" layer="96" rot="R90"/>
-</instance>
-<instance part="D1" gate="G$1" x="312.42" y="104.14" smashed="yes">
-<attribute name="NAME" x="309.88" y="101.6" size="1.27" layer="95"/>
-<attribute name="VALUE" x="313.69" y="86.36" size="1.27" layer="96" rot="R90"/>
+</instance>
+<instance part="D1" gate="G$1" x="314.96" y="104.14" smashed="yes">
+<attribute name="NAME" x="312.42" y="101.6" size="1.27" layer="95"/>
 </instance>
 <instance part="F2" gate="G$1" x="322.58" y="104.14"/>
@@
 <attribute name="VALUE" x="281.94" y="103.505" size="1.778" layer="96" rot="R180"/>
 </instance>
-<instance part="GND48" gate="1" x="279.4" y="66.04"/>
+<instance part="GND48" gate="1" x="274.32" y="66.04"/>
 <instance part="U$8" gate="G$1" x="302.26" y="170.18"/>
+<instance part="JP3" gate="G$1" x="241.3" y="38.1"/>
 </instances>
 <busses>
@@
 </segment>
 <segment>
-<wire x1="30.48" y1="48.26" x2="40.64" y2="48.26" width="0.1524" layer="91"/>
 <wire x1="40.64" y1="48.26" x2="45.72" y2="48.26" width="0.1524" layer="91"/>
 <pinref part="C9" gate="G$1" pin="2"/>
-<junction x="40.64" y="48.26"/>
-<pinref part="C11" gate="G$1" pin="2"/>
-<pinref part="C8" gate="G$1" pin="2"/>
 <pinref part="C10" gate="G$1" pin="2"/>
 <wire x1="45.72" y1="48.26" x2="50.8" y2="48.26" width="0.1524" layer="91"/>
-<wire x1="50.8" y1="48.26" x2="60.96" y2="48.26" width="0.1524" layer="91"/>
-<junction x="50.8" y="48.26"/>
 <pinref part="GND32" gate="1" pin="GND"/>
 <junction x="45.72" y="48.26"/>
@@
 <segment>
 <pinref part="GND46" gate="1" pin="GND"/>
-<wire x1="332.74" y1="96.52" x2="332.74" y2="88.9" width="0.1524" layer="91"/>
 <pinref part="D4" gate="G$1" pin="A"/>
 </segment>
@@
 <pinref part="JP1" gate="G$1" pin="1"/>
 <pinref part="GND48" gate="1" pin="GND"/>
+<wire x1="274.32" y1="71.12" x2="274.32" y2="68.58" width="0.1524" layer="91"/>
+<pinref part="R13" gate="G$1" pin="1"/>
 <wire x1="274.32" y1="71.12" x2="279.4" y2="71.12" width="0.1524" layer="91"/>
-<wire x1="279.4" y1="71.12" x2="279.4" y2="68.58" width="0.1524" layer="91"/>
-<pinref part="R13" gate="G$1" pin="1"/>
-<wire x1="279.4" y1="71.12" x2="284.48" y2="71.12" width="0.1524" layer="91"/>
-<junction x="279.4" y="71.12"/>
+<junction x="274.32" y="71.12"/>
 </segment>
 </net>
@@
 <wire x1="332.74" y1="104.14" x2="332.74" y2="101.6" width="0.1524" layer="91"/>
 <junction x="332.74" y="104.14"/>
-<wire x1="332.74" y1="104.14" x2="350.52" y2="104.14" width="0.1524" layer="91"/>
+<wire x1="332.74" y1="104.14" x2="337.82" y2="104.14" width="0.1524" layer="91"/>
 </segment>
 <segment>
@@
 </segment>
 <segment>
-<wire x1="30.48" y1="55.88" x2="40.64" y2="55.88" width="0.1524" layer="91"/>
 <wire x1="40.64" y1="55.88" x2="45.72" y2="55.88" width="0.1524" layer="91"/>
 <wire x1="45.72" y1="55.88" x2="50.8" y2="55.88" width="0.1524" layer="91"/>
@@
 <pinref part="P+6" gate="1" pin="V+"/>
 <pinref part="C9" gate="G$1" pin="1"/>
-<junction x="40.64" y="55.88"/>
-<pinref part="C11" gate="G$1" pin="1"/>
-<pinref part="C8" gate="G$1" pin="1"/>
 <pinref part="C10" gate="G$1" pin="1"/>
-<wire x1="50.8" y1="55.88" x2="60.96" y2="55.88" width="0.1524" layer="91"/>
-<junction x="50.8" y="55.88"/>
 </segment>
 <segment>
@@
 <segment>
 <pinref part="R13" gate="G$1" pin="2"/>
-<wire x1="294.64" y1="71.12" x2="297.18" y2="71.12" width="0.1524" layer="91"/>
-<wire x1="297.18" y1="71.12" x2="297.18" y2="73.66" width="0.1524" layer="91"/>
+<wire x1="289.56" y1="71.12" x2="292.1" y2="71.12" width="0.1524" layer="91"/>
+<wire x1="292.1" y1="71.12" x2="292.1" y2="73.66" width="0.1524" layer="91"/>
 <pinref part="R10" gate="G$1" pin="2"/>
-<wire x1="297.18" y1="73.66" x2="294.64" y2="73.66" width="0.1524" layer="91"/>
-<wire x1="297.18" y1="73.66" x2="299.72" y2="73.66" width="0.1524" layer="91"/>
-<junction x="297.18" y="73.66"/>
-<label x="299.72" y="73.66" size="1.27" layer="95" xref="yes"/>
+<wire x1="292.1" y1="73.66" x2="289.56" y2="73.66" width="0.1524" layer="91"/>
+<wire x1="292.1" y1="73.66" x2="294.64" y2="73.66" width="0.1524" layer="91"/>
+<junction x="292.1" y="73.66"/>
+<label x="294.64" y="73.66" size="1.27" layer="95" xref="yes"/>
 <wire x1="223.52" y1="147.32" x2="226.06" y2="147.32" width="0.1524" layer="91"/>
 <label x="226.06" y="147.32" size="1.27" layer="95" xref="yes"/>
@@
 <pinref part="F2" gate="G$1" pin="1"/>
 <pinref part="D1" gate="G$1" pin="C"/>
-<wire x1="317.5" y1="104.14" x2="314.96" y2="104.14" width="0.1524" layer="91"/>
 </segment>
 </net>
@@
 <net name="V_IN" class="0">
 <segment>
-<wire x1="307.34" y1="104.14" x2="309.88" y2="104.14" width="0.1524" layer="91"/>
-<label x="307.34" y="104.14" size="1.27" layer="95" rot="R180" xref="yes"/>
+<wire x1="309.88" y1="104.14" x2="312.42" y2="104.14" width="0.1524" layer="91"/>
+<label x="309.88" y="104.14" size="1.27" layer="95" rot="R180" xref="yes"/>
 <pinref part="D1" gate="G$1" pin="A"/>
 </segment>
@@
 <pinref part="JP1" gate="G$1" pin="2"/>
 <pinref part="R10" gate="G$1" pin="1"/>
-<wire x1="274.32" y1="73.66" x2="284.48" y2="73.66" width="0.1524" layer="91"/>
-</segment>
-</net>
+<wire x1="274.32" y1="73.66" x2="279.4" y2="73.66" width="0.1524" layer="91"/>
+</segment>
+</net>

Commit message: Organizing the schematic, small modifications to the PCB.
Parts:
- IC1: value PIC24FJ64GA002_QFN -> PIC24EP128GP202_QFN
Other:
- note added: "Battery monitor"
- note added: "GPS"
- note added: "In Circuit Serial Programming"
- note added: "Power Input"
- note added: "RC Output"
- note removed: "RC Out and Power In"
